File: jrgbwww24.sch (KiCad schematic (older format))
At the start: 28 parts, among them J1 Srew_terminal, J2 Screw_Terminal_01x06, Q1 2N3904, Q10 IPA040N06N, Q2 2N3904, Q3 2N3904, Q4 IPA040N06N, Q5 IPA040N06N, Q6 IPA040N06N, Q7 2N3904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

Commit message: some footprints
Parts:
- C1, C2: footprint (none) -> Capacitor_THT:CP_Radial_D5.0mm_P2.00mm
- D1, D2, D3: footprint (none) -> LED_SMD:LED_1206_3216Metric
- J1: footprint (none) -> TerminalBlock:TerminalBlock_bornier-2_P5.08mm
- J2: footprint (none) -> TerminalBlock:TerminalBlock_bornier-6_P5.08mm
- Q10, Q4, Q5, Q6, Q9: footprint Package_TO_SOT_SMD:TO-263-6 -> Package_TO_SOT_THT:TO-220F-3_Horizontal_TabDown
- R1: footprint Resistor_THT:R_Box_L8.4mm_W2.5mm_P5.08mm -> Resistor_THT:R_Axial_DIN0207_L6.3mm_D2.5mm_P7.62mm_Horizontal
- R2, R3, R4, R5, R6, R7, R8: footprint (none) -> Resistor_THT:R_Axial_DIN0207_L6.3mm_D2.5mm_P7.62mm_Horizontal
- SW1: footprint (none) -> jrgbwww24:1P2T SPDT
- U1: footprint (none) -> jrgbwww24:KeeYees ESP8266 ESP-12E
- U2: footprint (none) -> Package_TO_SOT_THT:TO-220-3_Horizontal_TabDown
Changed lines of the file:
@@
 F 0 "U1" H 2625 5165 50  0000 C CNN
 F 1 "esp8266" H 2625 5074 50  0000 C CNN
-F 2 "" H 2650 3850 50  0001 C CNN
+F 2 "jrgbwww24:KeeYees ESP8266 ESP-12E" H 2650 3850 50  0001 C CNN
 F 3 "" H 2650 3850 50  0001 C CNN
 	1    2650 3950
@@
 F 0 "C2" H 3765 1946 50  0000 L CNN
 F 1 "0.1u" H 3765 1855 50  0000 L CNN
-F 2 "" H 3688 1750 50  0001 C CNN
+F 2 "Capacitor_THT:CP_Radial_D5.0mm_P2.00mm" H 3688 1750 50  0001 C CNN
 F 3 "~" H 3650 1900 50  0001 C CNN
 	1    3650 1900
@@
 F 0 "C1" H 2435 1854 50  0000 R CNN
 F 1 "0.33u" H 2435 1945 50  0000 R CNN
-F 2 "" H 2588 1750 50  0001 C CNN
+F 2 "Capacitor_THT:CP_Radial_D5.0mm_P2.00mm" H 2588 1750 50  0001 C CNN
 F 3 "~" H 2550 1900 50  0001 C CNN
 	1    2550 1900
@@
 F 0 "R1" H 4630 2154 50  0000 R CNN
 F 1 "10K" H 4630 2245 50  0000 R CNN
-F 2 "Resistor_THT:R_Box_L8.4mm_W2.5mm_P5.08mm" V 4630 2200 50  0001 C CNN
+F 2 "Resistor_THT:R_Axial_DIN0207_L6.3mm_D2.5mm_P7.62mm_Horizontal" V 4630 2200 50  0001 C CNN
 F 3 "~" H 4700 2200 50  0001 C CNN
 	1    4700 2200
@@
 F 0 "SW1" H 2150 1900 50  0000 C CNN
 F 1 "SW_SPDT" H 2250 1800 50  0000 C CNN
-F 2 "" H 2100 1600 50  0001 C CNN
+F 2 "jrgbwww24:1P2T SPDT" H 2100 1600 50  0001 C CNN
 F 3 "~" H 2100 1600 50  0001 C CNN
 	1    2100 1600
@@
 F 0 "D1" H 7800 5550 50  0000 C CNN
 F 1 "RED - ALWAY ON" H 7950 5850 50  0000 C CNN
-F 2 "" H 7800 5700 50  0001 C CNN
+F 2 "LED_SMD:LED_1206_3216Metric" H 7800 5700 50  0001 C CNN
 F 3 "~" H 7800 5700 50  0001 C CNN
 	1    7800 5700
@@
 F 0 "J2" H 10130 3592 50  0000 L CNN
 F 1 "Screw_Terminal_01x06" H 10130 3501 50  0000 L CNN
-F 2 "" H 10050 3600 50  0001 C CNN
+F 2 "TerminalBlock:TerminalBlock_bornier-6_P5.08mm" H 10050 3600 50  0001 C CNN
 F 3 "~" H 10050 3600 50  0001 C CNN
 	1    10050 3600
@@
 F 0 "U2" H 3100 1649 50  0000 C CNN
 F 1 "L7805" H 3100 1740 50  0000 C CNN
-F 2 "" H 3125 1350 50  0001 L CIN
+F 2 "Package_TO_SOT_THT:TO-220-3_Horizontal_TabDown" H 3125 1350 50  0001 L CIN
 F 3 "http://www.st.com/content/ccc/resource/technical/document/datasheet/41/4f/b3/b0/12/d4/47/88/CD00000444.pdf/files/CD00000444.pdf/jcr:content/translations/en.CD00000444.pdf" H 3100 1450 50  0001 C CNN
 	1    3100 1500
@@
 F 0 "Q4" H 5604 2546 50  0000 L CNN
 F 1 "IPA040N06N" H 5600 2350 50  0000 L CNN
-F 2 "Package_TO_SOT_SMD:TO-263-6" H 5600 2425 50  0001 L CIN
+F 2 "Package_TO_SOT_THT:TO-220F-3_Horizontal_TabDown" H 5600 2425 50  0001 L CIN
 F 3 "https://www.infineon.com/dgdl/Infineon-IPB180N10S4_02-DS-v01_00-en.pdf?fileId=db3a30433d1d0bbe013d2129cf8a2f88" V 5400 2500 50  0001 L CNN
 	1    5400 2500
@@
 F 0 "R2" H 4630 3654 50  0000 R CNN
 F 1 "10K" H 4630 3745 50  0000 R CNN
-F 2 "" V 4630 3700 50  0001 C CNN
+F 2 "Resistor_THT:R_Axial_DIN0207_L6.3mm_D2.5mm_P7.62mm_Horizontal" V 4630 3700 50  0001 C CNN
 F 3 "~" H 4700 3700 50  0001 C CNN
 	1    4700 3700
@@
 F 0 "Q5" H 5604 4046 50  0000 L CNN
 F 1 "IPA040N06N" H 5600 3850 50  0000 L CNN
-F 2 "Package_TO_SOT_SMD:TO-263-6" H 5600 3925 50  0001 L CIN
+F 2 "Package_TO_SOT_THT:TO-220F-3_Horizontal_TabDown" H 5600 3925 50  0001 L CIN
 F 3 "https://www.infineon.com/dgdl/Infineon-IPB180N10S4_02-DS-v01_00-en.pdf?fileId=db3a30433d1d0bbe013d2129cf8a2f88" V 5400 4000 50  0001 L CNN
 	1    5400 4000
@@
 F 0 "R3" H 4630 5104 50  0000 R CNN
 F 1 "10K" H 4630 5195 50  0000 R CNN
-F 2 "" V 4630 5150 50  0001 C CNN
+F 2 "Resistor_THT:R_Axial_DIN0207_L6.3mm_D2.5mm_P7.62mm_Horizontal" V 4630 5150 50  0001 C CNN
 F 3 "~" H 4700 5150 50  0001 C CNN
 	1    4700 5150
@@
 F 0 "Q6" H 5604 5496 50  0000 L CNN
 F 1 "IPA040N06N" H 5600 5300 50  0000 L CNN
-F 2 "Package_TO_SOT_SMD:TO-263-6" H 5600 5375 50  0001 L CIN
+F 2 "Package_TO_SOT_THT:TO-220F-3_Horizontal_TabDown" H 5600 5375 50  0001 L CIN
 F 3 "https://www.infineon.com/dgdl/Infineon-IPB180N10S4_02-DS-v01_00-en.pdf?fileId=db3a30433d1d0bbe013d2129cf8a2f88" V 5400 5450 50  0001 L CNN
 	1    5400 5450
@@
 F 0 "R4" H 7330 2104 50  0000 R CNN
 F 1 "10K" H 7330 2195 50  0000 R CNN
-F 2 "" V 7330 2150 50  0001 C CNN
+F 2 "Resistor_THT:R_Axial_DIN0207_L6.3mm_D2.5mm_P7.62mm_Horizontal" V 7330 2150 50  0001 C CNN
 F 3 "~" H 7400 2150 50  0001 C CNN
 	1    7400 2150
@@
 F 0 "Q9" H 8304 2496 50  0000 L CNN
 F 1 "IPA040N06N" H 8300 2300 50  0000 L CNN
-F 2 "Package_TO_SOT_SMD:TO-263-6" H 8300 2375 50  0001 L CIN
+F 2 "Package_TO_SOT_THT:TO-220F-3_Horizontal_TabDown" H 8300 2375 50  0001 L CIN
 F 3 "https://www.infineon.com/dgdl/Infineon-IPB180N10S4_02-DS-v01_00-en.pdf?fileId=db3a30433d1d0bbe013d2129cf8a2f88" V 8100 2450 50  0001 L CNN
 	1    8100 2450
@@
 F 0 "R5" H 7330 3604 50  0000 R CNN
 F 1 "10K" H 7330 3695 50  0000 R CNN
-F 2 "" V 7330 3650 50  0001 C CNN
+F 2 "Resistor_THT:R_Axial_DIN0207_L6.3mm_D2.5mm_P7.62mm_Horizontal" V 7330 3650 50  0001 C CNN
 F 3 "~" H 7400 3650 50  0001 C CNN
 	1    7400 3650
@@
 F 0 "Q10" H 8304 3996 50  0000 L CNN
 F 1 "IPA040N06N" H 8300 3800 50  0000 L CNN
-F 2 "Package_TO_SOT_SMD:TO-263-6" H 8300 3875 50  0001 L CIN
+F 2 "Package_TO_SOT_THT:TO-220F-3_Horizontal_TabDown" H 8300 3875 50  0001 L CIN
 F 3 "https://www.infineon.com/dgdl/Infineon-IPB180N10S4_02-DS-v01_00-en.pdf?fileId=db3a30433d1d0bbe013d2129cf8a2f88" V 8100 3950 50  0001 L CNN
 	1    8100 3950
@@
 F 0 "D2" H 8500 5550 50  0000 C CNN
 F 1 "YELLOW - 5V" H 8650 5850 50  0000 C CNN
-F 2 "" H 8500 5700 50  0001 C CNN
+F 2 "LED_SMD:LED_1206_3216Metric" H 8500 5700 50  0001 C CNN
 F 3 "~" H 8500 5700 50  0001 C CNN
 	1    8500 5700
@@
 F 0 "R7" V 8293 5400 50  0000 C CNN
 F 1 "125" V 8384 5400 50  0000 C CNN
-F 2 "" V 8430 5400 50  0001 C CNN
+F 2 "Resistor_THT:R_Axial_DIN0207_L6.3mm_D2.5mm_P7.62mm_Horizontal" V 8430 5400 50  0001 C CNN
 F 3 "~" H 8500 5400 50  0001 C CNN
 	1    8500 5400
@@
 F 0 "D3" H 9200 5550 50  0000 C CNN
 F 1 "BLUE - 24V" H 9350 5850 50  0000 C CNN
-F 2 "" H 9200 5700 50  0001 C CNN
+F 2 "LED_SMD:LED_1206_3216Metric" H 9200 5700 50  0001 C CNN
 F 3 "~" H 9200 5700 50  0001 C CNN
 	1    9200 5700
@@
 F 0 "R8" V 8993 5400 50  0000 C CNN
 F 1 "1.05K" V 9084 5400 50  0000 C CNN
-F 2 "" V 9130 5400 50  0001 C CNN
+F 2 "Resistor_THT:R_Axial_DIN0207_L6.3mm_D2.5mm_P7.62mm_Horizontal" V 9130 5400 50  0001 C CNN
 F 3 "~" H 9200 5400 50  0001 C CNN
 	1    9200 5400
@@
 F 0 "R6" V 7593 5400 50  0000 C CNN
 F 1 "1.1K" V 7684 5400 50  0000 C CNN
-F 2 "" V 7730 5400 50  0001 C CNN
+F 2 "Resistor_THT:R_Axial_DIN0207_L6.3mm_D2.5mm_P7.62mm_Horizontal" V 7730 5400 50  0001 C CNN
 F 3 "~" H 7800 5400 50  0001 C CNN
 	1    7800 5400
@@
 F 0 "J1" H 1700 1650 50  0000 C CNN
 F 1 "Srew_terminal" H 1850 1750 50  0000 C CNN
-F 2 "" H 1500 1700 50  0001 C CNN
+F 2 "TerminalBlock:TerminalBlock_bornier-2_P5.08mm" H 1500 1700 50  0001 C CNN
 F 3 "~" H 1500 1700 50  0001 C CNN
 	1    1500 1700

Commit message: traces!
Parts:
- Q10, Q4, Q5, Q6, Q9: footprint Package_TO_SOT_THT:TO-220F-3_Horizontal_TabDown -> Package_TO_SOT_THT:TO-220F-3_Vertical
Connections:
- net +24V: no longer J1.2 (Pin_2), R6.2, SW1.2 (B)
- new net VDD: J1.2 (Pin_2), R6.2, SW1.2 (B)
Changed lines of the file:
@@
 WW_GND
-$Comp
-L power:+24V #24V0101
-U 1 1 617213A1
-P 1800 1400
-F 0 "#24V0101" H 1800 1250 50  0001 C CNN
-F 1 "+24V" H 1815 1573 50  0000 C CNN
-F 2 "" H 1800 1400 50  0001 C CNN
-F 3 "" H 1800 1400 50  0001 C CNN
-	1    1800 1400
-	1    0    0    -1
-$EndComp
 $Comp
 L Regulator_Linear:L7805 U2
@@
 F 0 "Q4" H 5604 2546 50  0000 L CNN
 F 1 "IPA040N06N" H 5600 2350 50  0000 L CNN
-F 2 "Package_TO_SOT_THT:TO-220F-3_Horizontal_TabDown" H 5600 2425 50  0001 L CIN
+F 2 "Package_TO_SOT_THT:TO-220F-3_Vertical" H 5600 2425 50  0001 L CIN
 F 3 "https://www.infineon.com/dgdl/Infineon-IPB180N10S4_02-DS-v01_00-en.pdf?fileId=db3a30433d1d0bbe013d2129cf8a2f88" V 5400 2500 50  0001 L CNN
 	1    5400 2500
@@
 F 0 "Q5" H 5604 4046 50  0000 L CNN
 F 1 "IPA040N06N" H 5600 3850 50  0000 L CNN
-F 2 "Package_TO_SOT_THT:TO-220F-3_Horizontal_TabDown" H 5600 3925 50  0001 L CIN
+F 2 "Package_TO_SOT_THT:TO-220F-3_Vertical" H 5600 3925 50  0001 L CIN
 F 3 "https://www.infineon.com/dgdl/Infineon-IPB180N10S4_02-DS-v01_00-en.pdf?fileId=db3a30433d1d0bbe013d2129cf8a2f88" V 5400 4000 50  0001 L CNN
 	1    5400 4000
@@
 F 0 "Q6" H 5604 5496 50  0000 L CNN
 F 1 "IPA040N06N" H 5600 5300 50  0000 L CNN
-F 2 "Package_TO_SOT_THT:TO-220F-3_Horizontal_TabDown" H 5600 5375 50  0001 L CIN
+F 2 "Package_TO_SOT_THT:TO-220F-3_Vertical" H 5600 5375 50  0001 L CIN
 F 3 "https://www.infineon.com/dgdl/Infineon-IPB180N10S4_02-DS-v01_00-en.pdf?fileId=db3a30433d1d0bbe013d2129cf8a2f88" V 5400 5450 50  0001 L CNN
 	1    5400 5450
@@
 F 0 "Q9" H 8304 2496 50  0000 L CNN
 F 1 "IPA040N06N" H 8300 2300 50  0000 L CNN
-F 2 "Package_TO_SOT_THT:TO-220F-3_Horizontal_TabDown" H 8300 2375 50  0001 L CIN
+F 2 "Package_TO_SOT_THT:TO-220F-3_Vertical" H 8300 2375 50  0001 L CIN
 F 3 "https://www.infineon.com/dgdl/Infineon-IPB180N10S4_02-DS-v01_00-en.pdf?fileId=db3a30433d1d0bbe013d2129cf8a2f88" V 8100 2450 50  0001 L CNN
 	1    8100 2450
@@
 F 0 "Q10" H 8304 3996 50  0000 L CNN
 F 1 "IPA040N06N" H 8300 3800 50  0000 L CNN
-F 2 "Package_TO_SOT_THT:TO-220F-3_Horizontal_TabDown" H 8300 3875 50  0001 L CIN
+F 2 "Package_TO_SOT_THT:TO-220F-3_Vertical" H 8300 3875 50  0001 L CIN
 F 3 "https://www.infineon.com/dgdl/Infineon-IPB180N10S4_02-DS-v01_00-en.pdf?fileId=db3a30433d1d0bbe013d2129cf8a2f88" V 8100 3950 50  0001 L CNN
 	1    8100 3950
@@
 $EndComp
 $Comp
-L power:+24V #24Volt0105
-U 1 1 614CA67E
-P 7800 5100
-F 0 "#24Volt0105" H 7800 4950 50  0001 C CNN
-F 1 "+24V" H 7815 5273 50  0000 C CNN
-F 2 "" H 7800 5100 50  0001 C CNN
-F 3 "" H 7800 5100 50  0001 C CNN
-	1    7800 5100
-	1    0    0    -1
-$EndComp
-$Comp
 L power:+24V #24Volt0106
 U 1 1 614CB3EF
@@
 	1    0    0    -1
 $EndComp
+$Comp
+L power:VDD #PWR0101
+U 1 1 616EC5C3
+P 1800 1400
+F 0 "#PWR0101" H 1800 1250 50  0001 C CNN
+F 1 "VDD" H 1815 1573 50  0000 C CNN
+F 2 "" H 1800 1400 50  0001 C CNN
+F 3 "" H 1800 1400 50  0001 C CNN
+	1    1800 1400
+	1    0    0    -1
+$EndComp
+$Comp
+L power:VDD #PWR?
+U 1 1 6170ACFF
+P 7800 5100
+F 0 "#PWR?" H 7800 4950 50  0001 C CNN
+F 1 "VDD" H 7815 5273 50  0000 C CNN
+F 2 "" H 7800 5100 50  0001 C CNN
+F 3 "" H 7800 5100 50  0001 C CNN
+	1    7800 5100
+	1    0    0    -1
+$EndComp
